File: batteryCharger/batteryCharger.sch (EAGLE design)
At the start: 71 parts, among them J1 B4P-VH(LF)(SN), Q1 SIR414DP-T1-GE3, Q2 SI7635DP-T1-GE3, Q3 SI7635DP-T1-GE3, Q4 SIR414DP-T1-GE3, Q5 SI7635DP-T1-GE3

Commit message: final board file
Parts:
- added R21, R22, R23: (no value), pot:TRIM_EU-3223W
Connections:
- removed net N$11: R5.1, RN2B.2, TM1.A
- removed net N$9: R19.1, RN2A.2, TM3.A
- new net ACSET_TRIM: R19.1, R23.A, RN2A.2, TM3.A
- new net ISET1_TRIM: R21.A, R5.1, RN2B.2, TM1.A
- net ACSET: now also R23.S
- net GND: now also R21.E, R22.E, R23.E
- net ISET1: now also R21.S
- net ISET2: now also R22.S
- net VREF: now also R22.A
Other:
- moved on the sheet: RN2A, RN2B, TM1, TM2, TM3

Commit message: v2 with bug fixses
Parts:
- added R24: 10k, SparkFun-Resistors:RESISTOR0603
- renumbered D1 to CHARGING, D2 to DONE, D3 to PG
Connections:
- removed net N$19: C5.1, Q2.D, Q3.D, R8.1, RN2D.2
- new net N$11: C5.1, Q2.S, Q3.S, R8.1, RN2D.2
- net ADAPTER: now also Q2.D; no longer Q2.S
- net GND: now also R24.2
- net N$10: now also R24.1
- net N$13: now also Q3.D; no longer Q3.S
- net OUTPUT: now also Q5.S; no longer Q5.D
- net PACK: now also Q5.D; no longer Q5.S
Other:
- moved on the sheet: Q5

Commit message: Bug fixses
Parts:
- removed TP3, TP6: TPTP20SQ, testpad:TPTP20SQ
- added F2: SMD-MICRO-FUSE-BLOCK, f-lf-omniblok-s:SMD-MICRO-FUSE-BLOCK
- R10, R9: value 10mOhm -> 0.01
- R17: value 100k -> 18k
- R18: value 30k -> 22.1k
- R19, R5: value 10k -> 18k
- R4: value 30k -> 32.4k
Connections:
- net N$10 renamed CE
- net N$4 renamed STAT1
- net N$7 renamed STAT2
- net N$8 renamed PG
- removed net N$21: D4.C, U$1.BTST
- new net ISET2_TRIM: R17.1, R22.A, RN2C.2, TM2.A
- new net N$9: C9.2, D4.C, U$1.BTST
- new net PW: C14.2, C19.1, C20.1, C3.1, F2.2, Q1.D, Q5.S, R20.2, R9.2, U$1.ACN
- net GND: no longer TP6.TP
- net N$22: no longer C9.2
- net OUTPUT: now also F2.1; no longer C14.2, C19.1, C20.1, C3.1, Q1.D, Q5.S, R20.2, R9.2, TP3.TP, U$1.ACN
- net VREF: now also RN2C.1; no longer R17.1, R22.A, TM2.A
Other:
- moved on the sheet: C1, CHARGING, D4, D5, DONE, OK1, PG, Q6, RN1A, RN1B, RN2A, RN2B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

Commit message: Change the enable pin design
Parts:
- removed CN1: (no value), adafruit:JST_2PIN-SMT-RA
- removed D5: BAT60J, diode:BAT60J
- removed OK1: LTV816S, optocoupler:LTV816S
- removed Q6: (no value), semicon-smd-ipc:PNP-TRANSISTOR_SOT23
- removed R11, R24: 10k, SparkFun-Resistors:RESISTOR0603
- removed R15: 1.2k, SparkFun-Resistors:RESISTOR0603
- removed TP1, TP2, TP4, TP5: TPTP20SQ, testpad:TPTP20SQ
- removed TP7: TPTP06SQ, testpad:TPTP06SQ
- added CH_EN, CH_EN1: SM02B-GHS-TB_LF__SN_, SM02B-GHS-TB_LF__SN_:SM02B-GHS-TB_LF__SN_
- added EN: JUMPER-SMT_2_NO_SILK, SparkFun-Jumpers:JUMPER-SMT_2_NO_SILK
- added JP1: JUMPER-SMT_3_1-NC_TRACE_NO-SILK, SparkFun-Jumpers:JUMPER-SMT_3_1-NC_TRACE_NO-SILK
- added LSP1, LSP2: LSP10, solpad:LSP10
- added Q7: SIR414DP-T1-GE3, SIR414DP-T1-GE3:SIR414DP-T1-GE3
- added R25: 1.2k, SparkFun-Resistors:RESISTOR0603
- added R26: 100k, SparkFun-Resistors:RESISTOR0603
Connections:
- removed net N$16: D5.C, OK1.A, R15.1
- new net GND_IN: Q7.S, R26.1, XA1.1
- new net N$4: Q7.G, R25.2
- net ADAPTER: now also EN.1
- net CE: now also JP1.2; no longer Q6.C, R24.1
- net EN: now also EN.2, R25.1, R26.2; no longer R15.2, TP7.TP
- net GND: now also CH_EN.3, CH_EN.4, CH_EN1.2, CH_EN1.3, CH_EN1.4, LSP2.MP, Q7.D; no longer CN1.1, D5.A, OK1.C, OK1.EMIT, R24.2, TP2.TP, TP4.TP, XA1.1
- net INPUT: no longer TP5.TP
- net N$3: now also CH_EN.2, JP1.1; no longer OK1.COL, Q6.B, R11.1
- net PACK: no longer TP1.TP
- net TSEN: now also CH_EN1.1, LSP1.MP; no longer CN1.2
- net VREF: now also CH_EN.1, JP1.3; no longer Q6.E, R11.2
Other:
- moved on the sheet: CHARGING, DONE, PG, RN1A, RN1B, RN2A, RN2B, RN2C, TM1, TM2, TM3
